Commit message: changed color

File: bumperbot_description/urdf/bumperbot.urdf.xacro (robot description, xacro)
@@ -163,5 +163,5 @@
         <mesh filename="package://bumperbot_description/meshes/imu_link.STL" />
       </geometry>
-      <material name="blue"/>
+      <material name="red"/>
     </visual>
     <collision>
@@ -191,5 +191,5 @@
         <mesh filename="package://bumperbot_description/meshes/laser_link.STL" />
       </geometry>
-      <material name="dark_grey"/>
+      <material name="gold"/>
     </visual>
     <collision>
@@ -218,3 +218,9 @@
     <color rgba="0.3 0.3 0.3 1"/>
   </material>
+  <material name="gold">
+    <color rgba="1 0.84 0 1"/>
+  </material>
+  <material name="red">
+    <color rgba="1 0 0 1"/>
+  </material>
 </robot>
